Commit message: modify urdf files

File: urdf/manipulator/manipulator.urdf.xacro (robot description, xacro)
@@ -3,9 +3,9 @@
 <!--
     You can confirm your manipulator on "rviz" to put down this cord.
-    roslaunch urdf_tutorial display.launch model:=manipulator.urdf.xacro
+    roslaunch urdf_tutorial display.launch model:=urdf/manipulator/manipulator.urdf.xacro
 -->
-    <xacro:include filename="$(find manipulator_simulation)/urdf/manipulator_parts.xacro"/>
-    <!-- xacro:include filename="$(find manipulator_simulation)/urdf/camera.xacro"/-->
-    <xacro:include filename="$(find manipulator_simulation)/urdf/hand_parts.xacro"/>
+    <xacro:include filename="$(find manipulator_simulation)/urdf/manipulator/manipulator_parts.xacro"/>
+    <!-- xacro:include filename="$(find manipulator_simulation)/urdf/manipulator/camera.xacro"/-->
+    <xacro:include filename="$(find manipulator_simulation)/urdf/manipulator/hand_parts.xacro"/>
     <!-- define colors -->
     <material name = "black">
@@ -18,10 +18,10 @@
     <link name = "world"/>
     <xacro:property name = "end_effector_base_link" value = "wrist_base_link"/>
-    <xacro:manipulator parent = "world" end_effector_link = "${end_effector_base_link}"
-        link_colour_1 = "black" link_colour_2 = "grey">
+    <xacro:manipulator  parent = "world"        end_effector_link = "${end_effector_base_link}"
+                        link_colour_1 = "black" link_colour_2 = "grey">
         <!-- define position where we want to set manupulator in the original point of link "world" -->
         <origin xyz = "0 0 0" rpy = "0 0 0"/>
     </xacro:manipulator>
-    <xacro:gripper base_link_name = "${end_effector_base_link}"
-        base_colour = "black" finger_colour = "grey"/>
+    <xacro:gripper  base_link_name = "${end_effector_base_link}"
+                    base_colour = "black" finger_colour = "grey"/>
 </robot>

File: urdf/manipulator/manipulator_parts.xacro (robot description, xacro)
@@ -2,5 +2,5 @@
 <!--
     You can confirm your manipulator on "rviz" to put down this cord.
-    roslaunch urdf_tutorial display.launch model:=urdf/manipulator.urdf.xacro
+    roslaunch urdf_tutorial display.launch model:=urdf/manipulator/manipulator.urdf.xacro
 -->
 <robot name = "manipulator" xmlns:xacro = "http://ros.org/wiki/xacro">
@@ -9,5 +9,5 @@
         params = "parent end_effector_link link_colour_1 link_colour_2 *origin">
         <!-- base -->
-        <xacro:property name = "PI" value = "3.14159"/>
+        <xacro:property name = "PI"     value = "3.14159"/>
         <xacro:property name = "BASE_X" value = "0.30"/>
         <xacro:property name = "BASE_Y" value = "0.30"/>
